File: stm32F1_dev_schematic.sch (EAGLE design)
At the start: 22 parts, among them IC1 AMS1117-3.3V, IC2 STM32F103C8T6, X1 MINI-USB-SCHIELD-32005-301

Commit message: board done routing
Parts:
- added R3: 1k5, SparkFun-Resistors:0.22OHM-0805-1/4W-1%
- added R4, R5: 2k2, SparkFun-Resistors:0.22OHM-0805-1/4W-1%
- added SV1: (no value), con-lstb:MA05-2
- added SV2, SV3: (no value), con-lstb:MA04-1
- added SV4, SV5: (no value), con-lstb:MA03-1
Connections:
- net HSE_OUT- renamed HSEOUT_N
- net USB-D+ renamed USB_P
- net USB-D- renamed USB_N
- removed net HSE_IN+: C12.2, C13.2, IC2.PD0-OSC_IN, L1.GND_1, L1.GND_2
- removed net N$2: C12.1, L1.CRYSTAL_1
- new net GI1: IC2.PB9, SV5.3
- new net GI2: IC2.PB8, SV5.2
- new net GI3: IC2.PB7, SV5.1
- new net GO1: IC2.PA3, SV4.3
- new net GO2: IC2.PA4, SV4.2
- new net GO3: IC2.PA5, SV4.1
- new net HSEIN_P: C12.1, IC2.PD0-OSC_IN, L1.CRYSTAL_1
- new net I2C2_SCL: IC2.PB10, R5.2, SV2.3
- new net I2C2_SDA: IC2.PB11, R4.2, SV2.2
- new net N$3: R3.2, SV1.2
- new net N$6: SV1.8
- new net SWCLK: IC2.PA14, SV1.4
- new net SWDIO: IC2.PA13, R3.1
- new net SWO: IC2.PB3, SV1.6
- new net USART_RX: IC2.PA10, SV3.2
- new net USART_TX: IC2.PA9, SV3.3
- net +3V3: now also R4.1, R5.1, SV1.1, SV2.4, SV3.4
- net GND: now also C12.2, C13.2, L1.GND_1, L1.GND_2, SV1.3, SV1.5, SV1.9, SV2.1, SV3.1
- net NRST: now also SV1.10
